Commit message: gazebo model_caster

File: src/winter_description/urdf/winter_gazebo.urdf.xacro (robot description, xacro)
@@ -9,13 +9,15 @@
         <xacro:property name="body_radius"      value=".25"/>
         <xacro:property name="body_height"      value=".127"/>
-	<xacro:property name="body_mass"   	value="0.7" />
+        <xacro:property name="body_mass"   	    value="0.7" />
         <xacro:property name="wheel_separation" value="${body_radius*2}"/>
         <xacro:property name="wheel_radius"     value=".075"/>
         <xacro:property name="wheel_length"     value=".06"/>
         <xacro:property name="wheel_color"      value="0 0 .8 1"/>
-	<xacro:property name="wheel_mass"   	value="0.4" />
+        <xacro:property name="wheel_mass"   	  value="0.4" />
+        <xacro:property name="caster_radius"    value="0.0325" />
+        <xacro:property name="caster_mass"      value="0.3" />
         <xacro:property name="laser_height"     value=".08"/>
         <xacro:property name="laser_radius"     value=".05"/>
-	<xacro:property name="laser_mass"   	value="0.2" />
+        <xacro:property name="laser_mass"   	  value="0.2" />
   <!-- Macro for inertia matrix -->
   <xacro:macro name="sphere_inertial_matrix" params="m r">
@@ -43,4 +45,34 @@
       </inertial>
   </xacro:macro>
+  <!-- Macro for caster joint --><!-- fb: front, back -->
+   <xacro:macro name="caster" params="fb caster_joint_origin_x">
+      <link name="caster_${fb}_link">
+          <visual>
+              <origin xyz="0 0 0" rpy="0 0 0" />
+              <geometry>
+                  <sphere radius="${caster_radius}" />
+              </geometry>
+              <material name="Black" />
+          </visual>
+          <collision>
+              <origin xyz="0 0 0" rpy="0 0 0 " />
+              <geometry>
+                  <sphere radius="${caster_radius}" />
+              </geometry>
+          </collision>
+          <sphere_inertial_matrix  m="${caster_mass}" r="${caster_radius}" />
+      </link>
+      <gazebo reference="caster_${fb}_link">
+          <material>Gazebo/Black</material>
+      </gazebo>
+      <joint name="base_to_caster_${fb}_joint" type="fixed">
+          <parent link="base_link"/>
+          <child link="caster_${fb}_link"/>
+          <origin xyz="${caster_joint_origin_x} 0 ${caster_radius}" rpy="0 0 0" />
+      </joint>
+        </xacro:macro>
+      <!-- caster Definitions -->
+      <caster fb="front"  caster_joint_origin_x="${body_radius}" />
+      <caster fb="back"  caster_joint_origin_x="-${body_radius}" />
 <!--base_link-->
         <link name="base_link">

Commit message: gazebo laser

File: src/winter_description/urdf/winter_gazebo.urdf.xacro (robot description, xacro)
@@ -2,5 +2,7 @@
 <robot xmlns:sensor="http://playerstage.sourceforge.net/gazebo/xmlschema/#sensor"
        xmlns:controller="http://playerstage.sourceforge.net/gazebo/xmlschema/#controller"
-       xmlns:xacro="http://www.ros.org/wiki/xacro" name="winter">
+       xmlns:interface="http://playerstage.sourceforge.net/gazebo/xmlschema/#interface"
+       xmlns:xacro="http://playerstage.sourceforge.net/gazebo/xmlschema/#interface"
+       name="winter">
 	<!-- sensors -->
   	<xacro:include filename="$(find winter_description)/urdf/sensors/hokuyo_urg04_laser.urdf.xacro"/>
@@ -95,5 +97,8 @@
   	</gazebo>
 <!--laser_link-->
-        <link name="laser_link">
+<xacro:hokuyo_urg04_laser name="base_laser_front" parent="base" ros_topic="scan_front" update_rate="10" min_angle="-1.57" max_angle="1.57">
+    <origin xyz="0 0 ${body_height+wheel_radius+0.04}" rpy="0 0 0"/>
+  </xacro:hokuyo_urg04_laser>
+        <!-- <link name="laser_link">
 	<cylinder_inertial_matrix  m="${laser_mass}" r="${laser_radius}" h="${laser_height}" />
                 <visual>
@@ -120,5 +125,5 @@
             <child link="laser_link"/>
             <origin xyz="0 0 ${body_height+wheel_radius}"/>
-        </joint>
+        </joint> -->
 <!-- left wheel-->
         <link name="left_wheel">

Commit message: navigation和gazebo 修正

File: src/winter_description/urdf/winter_gazebo.urdf.xacro (robot description, xacro)
@@ -77,4 +77,25 @@
       <caster fb="front"  caster_joint_origin_x="${body_radius}" />
       <caster fb="back"  caster_joint_origin_x="-${body_radius}" />
+      <!-- base_footprint -->
+      <link name="base_footprint">
+          <inertial>
+              <mass value="0.0001" />
+              <origin xyz="0 0 0" />
+              <inertia ixx="0.0001" ixy="0.0" ixz="0.0"
+                  iyy="0.0001" iyz="0.0"
+                  izz="0.0001" />
+          </inertial>
+          <visual>
+              <origin xyz="0 0 0" rpy="0 0 0" />
+              <geometry>
+                  <box size="0.001 0.001 0.001" />
+              </geometry>
+          </visual>
+      </link>
+      <joint name="base_footprint_joint" type="fixed">
+          <origin xyz="0 0 ${wheel_radius}" rpy="0 0 0" />
+          <parent link="base_footprint"/>
+          <child link="base_link" />
+      </joint>
 <!--base_link-->
         <link name="base_link">
@@ -205,5 +226,8 @@
       </transmission>
 <gazebo>
-    <plugin name="gazebo_ros_controller" filename="libgazebo_ros_control.so" />
+    <plugin name="gazebo_ros_controller" filename="libgazebo_ros_control.so" >
+      <robotNamespace>/</robotNamespace>
+      <robotSimType>gazebo_ros_control/DefaultRobotHWSim</robotSimType>
+    </plugin>
   </gazebo>
 </robot>

Commit message: navigation和gazebo topic 修正

File: src/winter_description/urdf/winter_gazebo.urdf.xacro (robot description, xacro)
@@ -120,33 +120,7 @@
 <xacro:hokuyo_urg04_laser name="base_laser_front" parent="base" ros_topic="scan_front" update_rate="10" min_angle="-3.14" max_angle="3.14">
     <origin xyz="0 0 ${body_height+wheel_radius+0.04}" rpy="0 0 0"/>
-  </xacro:hokuyo_urg04_laser>
-        <!-- <link name="laser_link">
-	<cylinder_inertial_matrix  m="${laser_mass}" r="${laser_radius}" h="${laser_height}" />
-                <visual>
-                        <geometry>
-                                <cylinder length="${laser_height}" radius="${laser_radius}"/>
-                        </geometry>
-                        <material name="green">
-                                <color rgba="0 0.8 0 1"/>
-                        </material>
-                        <origin xyz="0 0 ${laser_height/2}"/>
-                </visual>
-                <collision>
-                        <geometry>
-                                <cylinder length="${laser_height}" radius="${laser_radius}"/>
-                        </geometry>
-                        <origin xyz="0 0 ${laser_height/2}"/>
-                </collision>
-        </link>
-  <gazebo reference="laser_link">
-      <material>Gazebo/Black</material>
-  </gazebo>
-        <joint name="laser_link_to_base_link" type="fixed">
-            <parent link="base_link"/>
-            <child link="laser_link"/>
-            <origin xyz="0 0 ${body_height+wheel_radius}"/>
-        </joint> -->
+</xacro:hokuyo_urg04_laser>
 <!-- left wheel-->
-        <link name="left_wheel">
+<link name="left_wheel">
 	<cylinder_inertial_matrix  m="${wheel_mass}" r="${wheel_radius}" h="${wheel_length}" />
                 <visual>

Commit message: gazebo navigation v1.0

File: src/winter_description/urdf/winter_gazebo.urdf.xacro (robot description, xacro)
@@ -77,25 +77,4 @@
       <caster fb="front"  caster_joint_origin_x="${body_radius}" />
       <caster fb="back"  caster_joint_origin_x="-${body_radius}" />
-      <!-- base_footprint -->
-      <link name="base_footprint">
-          <inertial>
-              <mass value="0.0001" />
-              <origin xyz="0 0 0" />
-              <inertia ixx="0.0001" ixy="0.0" ixz="0.0"
-                  iyy="0.0001" iyz="0.0"
-                  izz="0.0001" />
-          </inertial>
-          <visual>
-              <origin xyz="0 0 0" rpy="0 0 0" />
-              <geometry>
-                  <box size="0.001 0.001 0.001" />
-              </geometry>
-          </visual>
-      </link>
-      <joint name="base_footprint_joint" type="fixed">
-          <origin xyz="0 0 ${wheel_radius}" rpy="0 0 0" />
-          <parent link="base_footprint"/>
-          <child link="base_link" />
-      </joint>
 <!--base_link-->
         <link name="base_link">
@@ -120,7 +99,33 @@
 <xacro:hokuyo_urg04_laser name="base_laser_front" parent="base" ros_topic="scan_front" update_rate="10" min_angle="-3.14" max_angle="3.14">
     <origin xyz="0 0 ${body_height+wheel_radius+0.04}" rpy="0 0 0"/>
-</xacro:hokuyo_urg04_laser>
+  </xacro:hokuyo_urg04_laser>
+        <!-- <link name="laser_link">
+	<cylinder_inertial_matrix  m="${laser_mass}" r="${laser_radius}" h="${laser_height}" />
+                <visual>
+                        <geometry>
+                                <cylinder length="${laser_height}" radius="${laser_radius}"/>
+                        </geometry>
+                        <material name="green">
+                                <color rgba="0 0.8 0 1"/>
+                        </material>
+                        <origin xyz="0 0 ${laser_height/2}"/>
+                </visual>
+                <collision>
+                        <geometry>
+                                <cylinder length="${laser_height}" radius="${laser_radius}"/>
+                        </geometry>
+                        <origin xyz="0 0 ${laser_height/2}"/>
+                </collision>
+        </link>
+  <gazebo reference="laser_link">
+      <material>Gazebo/Black</material>
+  </gazebo>
+        <joint name="laser_link_to_base_link" type="fixed">
+            <parent link="base_link"/>
+            <child link="laser_link"/>
+            <origin xyz="0 0 ${body_height+wheel_radius}"/>
+        </joint> -->
 <!-- left wheel-->
-<link name="left_wheel">
+        <link name="left_wheel">
 	<cylinder_inertial_matrix  m="${wheel_mass}" r="${wheel_radius}" h="${wheel_length}" />
                 <visual>
@@ -201,6 +206,10 @@
 <gazebo>
     <plugin name="gazebo_ros_controller" filename="libgazebo_ros_control.so" >
-      <robotNamespace>/</robotNamespace>
-      <robotSimType>gazebo_ros_control/DefaultRobotHWSim</robotSimType>
+	<robotNamespace>/</robotNamespace>
+      	<robotSimType>gazebo_ros_control/DefaultRobotHWSim</robotSimType>
+<commandTopic>cmd_vel</commandTopic>
+    <odometryTopic>odom</odometryTopic>
+    <odometryFrame>odom</odometryFrame>
+    <broadcastTF>true</broadcastTF>
     </plugin>
   </gazebo>

Commit message: move_base参数调整

File: src/winter_description/urdf/winter_gazebo.urdf.xacro (robot description, xacro)
@@ -77,6 +77,6 @@
       <caster fb="front"  caster_joint_origin_x="${body_radius}" />
       <caster fb="back"  caster_joint_origin_x="-${body_radius}" />
-<!--base_link-->
-        <link name="base_link">
+  <!--base_link-->
+	<link name="base_link">
 	<cylinder_inertial_matrix  m="${body_mass}" r="${body_radius}" h="${body_height}" />
                 <visual>
@@ -96,35 +96,9 @@
       		<material>Gazebo/White</material>
   	</gazebo>
-<!--laser_link-->
-<xacro:hokuyo_urg04_laser name="base_laser_front" parent="base" ros_topic="scan_front" update_rate="10" min_angle="-3.14" max_angle="3.14">
+  <!--laser_link-->
+  <xacro:hokuyo_urg04_laser name="base_laser_front" parent="base" ros_topic="scan_front" update_rate="10" min_angle="-3.14" max_angle="3.14">
     <origin xyz="0 0 ${body_height+wheel_radius+0.04}" rpy="0 0 0"/>
   </xacro:hokuyo_urg04_laser>
-        <!-- <link name="laser_link">
-	<cylinder_inertial_matrix  m="${laser_mass}" r="${laser_radius}" h="${laser_height}" />
-                <visual>
-                        <geometry>
-                                <cylinder length="${laser_height}" radius="${laser_radius}"/>
-                        </geometry>
-                        <material name="green">
-                                <color rgba="0 0.8 0 1"/>
-                        </material>
-                        <origin xyz="0 0 ${laser_height/2}"/>
-                </visual>
-                <collision>
-                        <geometry>
-                                <cylinder length="${laser_height}" radius="${laser_radius}"/>
-                        </geometry>
-                        <origin xyz="0 0 ${laser_height/2}"/>
-                </collision>
-        </link>
-  <gazebo reference="laser_link">
-      <material>Gazebo/Black</material>
-  </gazebo>
-        <joint name="laser_link_to_base_link" type="fixed">
-            <parent link="base_link"/>
-            <child link="laser_link"/>
-            <origin xyz="0 0 ${body_height+wheel_radius}"/>
-        </joint> -->
-<!-- left wheel-->
+  <!-- left wheel-->
         <link name="left_wheel">
 	<cylinder_inertial_matrix  m="${wheel_mass}" r="${wheel_radius}" h="${wheel_length}" />
@@ -154,5 +128,5 @@
                 <axis xyz="0 1 0"/>
         </joint>
-<!-- Transmission is important to link the joints and the controller -->
+  <!-- Transmission is important to link the joints and the controller -->
       <transmission name="wheel_left_joint_trans">
 		<type>transmission_interface/SimpleTransmission</type>
@@ -165,7 +139,7 @@
 		</actuator>
       </transmission>
-<!-- right wheel-->
+  <!-- right wheel-->
         <link name="right_wheel">
-<cylinder_inertial_matrix  m="${wheel_mass}" r="${wheel_radius}" h="${wheel_length}" />
+	<cylinder_inertial_matrix  m="${wheel_mass}" r="${wheel_radius}" h="${wheel_length}" />
                 <visual>
                         <geometry>
@@ -204,12 +178,12 @@
 		</actuator>
       </transmission>
-<gazebo>
+  <gazebo>
     <plugin name="gazebo_ros_controller" filename="libgazebo_ros_control.so" >
 	<robotNamespace>/</robotNamespace>
       	<robotSimType>gazebo_ros_control/DefaultRobotHWSim</robotSimType>
-<commandTopic>cmd_vel</commandTopic>
-    <odometryTopic>odom</odometryTopic>
-    <odometryFrame>odom</odometryFrame>
-    <broadcastTF>true</broadcastTF>
+	<commandTopic>cmd_vel</commandTopic>
+	<odometryTopic>odom</odometryTopic>
+	<odometryFrame>odom</odometryFrame>
+	<broadcastTF>true</broadcastTF>
     </plugin>
   </gazebo>
