Commit message: update clear_costmap_recovery

File: src/winter_simulation/urdf/moi_robot.urdf (robot description, URDF)
Before this commit: robot winter, 4 links, 3 joints
Links:
- added link ultrasound, mass 0.000001; visual box size=0.1 0.05 0.06
Joints:
- added joint ultronsonic: type fixed, parent base_link, child ultrasound, origin xyz=0.2 0.00 0.2 rpy=0 0 0

Commit message: update

File: src/winter_simulation/urdf/moi_robot.urdf (robot description, URDF)
Before this commit: robot winter, 5 links, 4 joints
Joints:
- joint left_wheel_to_base_link: origin xyz=0.0 0.25 0.075 -> xyz=0.0 0.20 0.075
- joint right_wheel_to_base_link: origin xyz=0.0 -0.25 0.075 -> xyz=0.0 -0.20 0.075

Commit message: update

File: src/winter_simulation/urdf/moi_robot.urdf (robot description, URDF)
Before this commit: robot winter, 5 links, 4 joints
Links:
- removed link laser_link
- added link base_laser_link; collision cylinder length=0.08 radius=0.05; visual cylinder length=0.08 radius=0.05
Joints:
- joint laser_link_to_base_link: child laser_link -> base_laser_link

Commit message: update winter_move_base

File: src/winter_simulation/urdf/moi_robot.urdf (robot description, URDF)
Before this commit: robot winter, 5 links, 4 joints
Links:
- added link camera_link; collision cylinder length=0.08 radius=0.05; visual cylinder length=0.08 radius=0.05
Joints:
- added joint kinect_link_to_base_link: type fixed, parent base_link, child camera_link, origin xyz=0 0 0.402

Commit message: update

File: src/winter_simulation/urdf/moi_robot.urdf (robot description, URDF)
Before this commit: robot winter, 6 links, 5 joints
Joints:
- joint laser_link_to_base_link: origin xyz=0 0 0.202 -> xyz=0.2 0 0.202
